File: hardware/squantlogger_chrome_hedgehog/squantlogger_chrome_hedgehog.kicad_pcb (KiCad board)
At the start: 2 copper layers, 93.9 x 59.9 mm, 8 parts, among them U1 USB-micro

Commit message: * started schematic of the chrome hedgehog board
Parts:
- removed C1: 100n, Capacitors_SMD:C_1206
- removed U1: USB-micro, SquantorUsb:SquantorUsb-USB-UB-SMD4H
- JP1, JP2: footprint SquantorConnectors:SquantorConnectors-2X18 -> SquantorConnectors:Header-0254-2X18-H010
Connections:
- net Earth renamed /Case_ground
