File: hardware/squantlogger_cobalt_ant/squantlogger_cobalt_ant.sch (KiCad schematic (older format))
At the start: 36 parts, among them J1 JTAG_2X05, J2 PINS_1X12, J3 PINS_1X12, U1 MCP1702-MB

Commit message: * added some more schematic connections to the breakout headers
Parts:
- added C? (x2): 18p, SquantorRcl:C_0402, symbol C
- added R? (x2): 10K, SquantorRcl:R_0402_hand, symbol R
- added R?: FERRITE, SquantorRcl:R_0805, symbol R
- added Y?: 12.0MHz, symbol Crystal
- M?: footprint SquantorNxp_SOT617-3 -> SquantorNxp:SOT617-3
- U?: footprint (none) -> SquantorWinbond:WINBOND_SS
Connections:
- net labels added: GPIO_0_1, GPIO_0_12, GPIO_0_15, GPIO_0_24, GPIO_0_28, GPIO_0_4, GPIO_12
- wire segments 100 -> 134
Other:
- moved on the sheet: C?, R?, U?

Commit message: * lots of smaller updates due to DRC errors * used powerjoiner component to connect analog and digital powerdomains * DAMN, not enough pins, I really need to get TQFP48 pin controller, but it is very large. Will need to switch to 4 copper layers :(
Parts:
- removed J2, J3: PINS_1X12, SquantorConnectors:Header-0254-1X12-H010, symbol PINS_1X12
- removed R?: FERRITE, SquantorRcl:R_0805, symbol R
- added C4: 1u, SquantorRcl:C_0402, symbol C
- added C5: 100n, SquantorRcl:C_0402, symbol C
- added J2: Cobalt_Ant_Digital, SquantorConnectors:Header-0254-1X12-H010, symbol Cobalt_Ant_Digital
- added J3: Cobalt_Ant_Analog, SquantorConnectors:Header-0254-1X12-H010, symbol Cobalt_Ant_Analog
- added R11: 33, SquantorRcl:R_0402_hand, symbol R
- added R6, R7: 10K, SquantorRcl:R_0402_hand, symbol R
- added U1, U2: POWER_JOINER, SquantorRcl:R_0805, symbol POWER_JOINER
- added U4: MCP1525, SquantorMicrochip:TT-(SOT23), symbol MCP1525
- J1: renamed from J?; footprint (none) -> SquantorConnectors:Header-0254-1X06-H010
- R18, R19: renamed from 2.2k; value R -> 2K2
- R22, R23: renamed from R?; footprint (none) -> SquantorRcl:R_0402_hand
- Y1: renamed from Y?; footprint (none) -> SquantorCrystal:X_5.0_3.2
- gave numbers to parts that had none: 13
- renumbered C2 to C1, C7 to C10, C1 to C2, C4 to C6, C5 to C7, C6 to C9, J1 to J4, R3 to R1, R2 to R10, R4 to R2, R5 to R3, R1 to R4, R7 to R5, R6 to R8, R8 to R9, U1 to U3
Connections:
- net ADC_0: now also J3.4 (ADC0)
- net ADC_1: now also J3.5 (ADC1)
- net ADC_2: now also J3.6 (ADC2)
- net ADC_3: now also J3.7 (ADC3)
- net ADC_4: now also J3.8 (ADC4)
- net ADC_5: now also J3.9 (ADC5)
- net ADC_6: now also J3.10 (ADC6)
- net ADC_7: now also M1.30 (ADC_7/PIO0_19), J3.11 (ADC7)
- net ADC_8: now also M1.31 (ADC_8/PIO0_18), J3.12 (ADC8)
- net GND: now also J2.1 (GND), U1.1 (IN)
- net GNDA: now also C4.2, C5.2, J3.1 (GNDA), U1.2 (OUT), U4.3 (GND)
- net GPIO_0_1: now also J2.10 (GPIO7)
- net GPIO_0_12: now also J2.3 (GPIO0)
- net GPIO_0_15: now also J2.9 (GPIO6)
- net GPIO_0_24: now also J2.8 (GPIO5)
- net GPIO_0_28: now also J2.5 (GPIO2)
- net GPIO_0_4: now also J2.4 (GPIO1)
- net I2C_SCL: now also J2.7 (GPIO4/SCL)
- net I2C_SDA: now also J2.6 (GPIO3/SDA)
- net VDD: now also J2.2 (VDD), R6.1, R7.1, U2.1 (IN)
- net VDDA: now also C5.1, J3.2 (VDDA), U2.2 (OUT), U4.1 (VIN)
- net VREF: now also C4.1, J3.3 (VREF), R11.2, U4.2 (VOUT); no longer M1.1 (PIO0_13/ADC10)
- new net: M1.1 (PIO0_13/ADC10), R11.1
- new net: J2.11 (GPIO8), R6.2
- new net: J2.12 (GPIO9), R7.2
Other:
- moved on the sheet: C1, C2, C3, U3
