File: hardware/squantlogger_nickel_beetle/nickel_beetle_breakout/nickel_beetle_breakout.kicad_pcb (KiCad board)
At the start: 4 copper layers, 44 x 29 mm, 6 parts, among them J1 Conn_02x10_Odd_Even, J2 Conn_02x10_Odd_Even

Commit message: DONE: nickel beetle gpio breakout
Parts:
- added J3: Conn_02x10_Odd_Even, SquantorConnectors:Header-0245-2X10-H010, F.Cu at (148.6, 97.8)
- added J4: Conn_02x10_Odd_Even, SquantorConnectors:Header-0245-2X10-H010, F.Cu at (148.6, 102.9)
- N2: value V20171120 -> V20180610
- moved N2 19.8 mm to (170.0, 100.0), turned to 90 degrees
- moved N1 15.4 mm to (165.7, 100.3), turned to 90 degrees
Connections:
- J1 pad 10: Net-(J1-Pad10) -> /ANALOG_05
- J1 pad 11: Net-(J1-Pad11) -> /ANALOG_06
- J1 pad 12: Net-(J1-Pad12) -> /ANALOG_07
- J1 pad 13: Net-(J1-Pad13) -> /ANALOG_08
- J1 pad 14: Net-(J1-Pad14) -> /ANALOG_09
- J1 pad 15: Net-(J1-Pad15) -> /ANALOG_10
- J1 pad 16: Net-(J1-Pad16) -> /ANALOG_11
- J1 pad 17: Net-(J1-Pad17) -> /ANALOG_12
- J1 pad 18: Net-(J1-Pad18) -> /ANALOG_13
- J1 pad 19: Net-(J1-Pad19) -> /ANALOG_14
- J1 pad 20: Net-(J1-Pad20) -> /ANALOG_15
- J1 pad 5: Net-(J1-Pad5) -> /ANALOG_00
- J1 pad 6: Net-(J1-Pad6) -> /ANALOG_01
- J1 pad 7: Net-(J1-Pad7) -> /ANALOG_02
- J1 pad 8: Net-(J1-Pad8) -> /ANALOG_03
- J1 pad 9: Net-(J1-Pad9) -> /ANALOG_04
- J2 pad 10: Net-(J2-Pad10) -> /DIGITAL_05
- J2 pad 11: Net-(J2-Pad11) -> /DIGITAL_06
- J2 pad 12: Net-(J2-Pad12) -> /DIGITAL_07
- J2 pad 13: Net-(J2-Pad13) -> /DIGITAL_08
- J2 pad 14: Net-(J2-Pad14) -> /DIGITAL_09
- J2 pad 15: Net-(J2-Pad15) -> /DIGITAL_10
- J2 pad 16: Net-(J2-Pad16) -> /DIGITAL_11
- J2 pad 17: Net-(J2-Pad17) -> /DIGITAL_12
- J2 pad 18: Net-(J2-Pad18) -> /DIGITAL_13
- J2 pad 19: Net-(J2-Pad19) -> /DIGITAL_14
- J2 pad 20: Net-(J2-Pad20) -> /DIGITAL_15
- J2 pad 5: Net-(J2-Pad5) -> /DIGITAL_00
- J2 pad 6: Net-(J2-Pad6) -> /DIGITAL_01
- J2 pad 7: Net-(J2-Pad7) -> /DIGITAL_02
- J2 pad 8: Net-(J2-Pad8) -> /DIGITAL_03
- J2 pad 9: Net-(J2-Pad9) -> /DIGITAL_04
Routing:
- net VDDA: track 0.00 -> 16.9 mm
- net VDD: track 0.00 -> 16.6 mm
- net VSSA: track 0.00 -> 15.1 mm
- net VSS: track 0.00 -> 14.7 mm
- net /ANALOG_14: track 0.00 -> 14.4 mm
- net /ANALOG_00: track 0.00 -> 13.9 mm
- net /ANALOG_12: track 0.00 -> 13.8 mm
- net /DIGITAL_15: track 0.00 -> 13.7 mm
- net /ANALOG_02: track 0.00 -> 13.4 mm
- net /ANALOG_10: track 0.00 -> 13.3 mm
- net /DIGITAL_13: track 0.00 -> 13.2 mm
- net /DIGITAL_01: track 0.00 -> 13.1 mm
- net /ANALOG_08: track 0.00 -> 13.0 mm
- net /ANALOG_04: track 0.00 -> 12.8 mm
- net /DIGITAL_03: track 0.00 -> 12.6 mm
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
Commit message: reworked nicked beetle breakout
Parts:
- J1, J2: footprint SquantorConnectors:Header_0127_2X10_H007 -> SquantorConnectors:Header-0127-2X10-H006
Routing:
- net /DIGITAL_15: track 13.7 -> 0.00 mm
- net /DIGITAL_13: track 13.2 -> 0.00 mm
- net /DIGITAL_01: track 13.1 -> 0.00 mm
- net /DIGITAL_03: track 12.6 -> 0.00 mm
- net /DIGITAL_11: track 12.6 -> 0.00 mm
- net /DIGITAL_05: track 12.1 -> 0.00 mm
- net /DIGITAL_09: track 12.1 -> 0.00 mm
- net /DIGITAL_07: track 11.6 -> 0.00 mm
- net /DIGITAL_14: track 8.83 -> 0.00 mm
- net /DIGITAL_00: track 8.83 -> 0.00 mm
- net /DIGITAL_02: track 8.30 -> 0.00 mm
- net /DIGITAL_12: track 8.30 -> 0.00 mm
- net /DIGITAL_10: track 7.77 -> 0.00 mm
- net /DIGITAL_04: track 7.77 -> 0.00 mm
- net /DIGITAL_08: track 7.25 -> 0.00 mm
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
Commit message: fixed PCB layout
Routing:
- net /DIGITAL_15: track 0.00 -> 12.4 mm
- net /DIGITAL_13: track 0.00 -> 11.9 mm
- net /DIGITAL_01: track 0.00 -> 11.4 mm
- net /DIGITAL_11: track 0.00 -> 11.4 mm
- net /DIGITAL_03: track 0.00 -> 10.8 mm
- net /DIGITAL_09: track 0.00 -> 10.8 mm
- net /DIGITAL_14: track 0.00 -> 10.6 mm
- net /DIGITAL_05: track 0.00 -> 10.3 mm
- net /DIGITAL_07: track 0.00 -> 10.3 mm
- net /DIGITAL_12: track 0.00 -> 10.1 mm
- net /DIGITAL_00: track 0.00 -> 10.1 mm
- net /DIGITAL_02: track 0.00 -> 9.57 mm
- net /DIGITAL_10: track 0.00 -> 9.57 mm
- net /DIGITAL_04: track 0.00 -> 9.04 mm
- net /DIGITAL_08: track 0.00 -> 9.02 mm
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Changed lines of the file:
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@@
     (thickness 1.6)
     (drawings 10)
-    (tracks 93)
+    (tracks 158)
     (zones 0)
     (modules 8)
@@
   (segment (start 156.25 88.30089) (end 156.25 91.3) (width 0.2) (layer F.Cu) (net 20))
   (segment (start 155.575 87.62589) (end 156.25 88.30089) (width 0.2) (layer F.Cu) (net 20))
+  (segment (start 146.05 109.3) (end 142.24 105.49) (width 0.2) (layer F.Cu) (net 21))
+  (segment (start 142.24 105.49) (end 142.24 104.14) (width 0.2) (layer F.Cu) (net 21))
+  (segment (start 146.05 111.75589) (end 146.05 109.3) (width 0.2) (layer F.Cu) (net 21))
+  (segment (start 146.685 112.39089) (end 146.05 111.75589) (width 0.2) (layer F.Cu) (net 21))
+  (segment (start 143.5 105.5) (end 143.5 102.86) (width 0.2) (layer F.Cu) (net 22))
+  (segment (start 143.5 102.86) (end 142.24 101.6) (width 0.2) (layer F.Cu) (net 22))
+  (segment (start 146.685 108.685) (end 143.5 105.5) (width 0.2) (layer F.Cu) (net 22))
+  (segment (start 146.685 111.12089) (end 146.685 108.685) (width 0.2) (layer F.Cu) (net 22))
+  (segment (start 147.3 108) (end 144.78 105.48) (width 0.2) (layer F.Cu) (net 23))
+  (segment (start 144.78 105.48) (end 144.78 104.14) (width 0.2) (layer F.Cu) (net 23))
+  (segment (start 147.3 111.73589) (end 147.3 108) (width 0.2) (layer F.Cu) (net 23))
+  (segment (start 147.955 112.39089) (end 147.3 111.73589) (width 0.2) (layer F.Cu) (net 23))
+  (segment (start 146.05 105.55) (end 146.05 102.87) (width 0.2) (layer F.Cu) (net 24))
+  (segment (start 146.05 102.87) (end 144.78 101.6) (width 0.2) (layer F.Cu) (net 24))
+  (segment (start 147.955 107.455) (end 146.05 105.55) (width 0.2) (layer F.Cu) (net 24))
+  (segment (start 147.955 111.12089) (end 147.955 107.455) (width 0.2) (layer F.Cu) (net 24))
+  (segment (start 148.6 106.75) (end 147.32 105.47) (width 0.2) (layer F.Cu) (net 25))
+  (segment (start 147.32 105.47) (end 147.32 104.14) (width 0.2) (layer F.Cu) (net 25))
+  (segment (start 148.6 111.76589) (end 148.6 106.75) (width 0.2) (layer F.Cu) (net 25))
+  (segment (start 149.225 112.39089) (end 148.6 111.76589) (width 0.2) (layer F.Cu) (net 25))
+  (segment (start 148.6 105.45) (end 148.6 102.88) (width 0.2) (layer F.Cu) (net 26))
+  (segment (start 148.6 102.88) (end 147.32 101.6) (width 0.2) (layer F.Cu) (net 26))
+  (segment (start 149.225 106.075) (end 148.6 105.45) (width 0.2) (layer F.Cu) (net 26))
+  (segment (start 149.225 111.12089) (end 149.225 106.075) (width 0.2) (layer F.Cu) (net 26))
+  (segment (start 149.85 111.75) (end 149.85 104.15) (width 0.2) (layer F.Cu) (net 27))
+  (segment (start 149.85 104.15) (end 149.86 104.14) (width 0.2) (layer F.Cu) (net 27))
+  (segment (start 150.49089 112.39089) (end 149.85 111.75) (width 0.2) (layer F.Cu) (net 27))
+  (segment (start 150.495 112.39089) (end 150.49089 112.39089) (width 0.2) (layer F.Cu) (net 27))
+  (segment (start 151.1 105.55) (end 151.1 102.84) (width 0.2) (layer F.Cu) (net 28))
+  (segment (start 151.1 102.84) (end 149.86 101.6) (width 0.2) (layer F.Cu) (net 28))
+  (segment (start 150.495 106.155) (end 151.1 105.55) (width 0.2) (layer F.Cu) (net 28))
+  (segment (start 150.495 111.12089) (end 150.495 106.155) (width 0.2) (layer F.Cu) (net 28))
+  (segment (start 151.15 106.7) (end 152.4 105.45) (width 0.2) (layer F.Cu) (net 29))
+  (segment (start 152.4 105.45) (end 152.4 104.14) (width 0.2) (layer F.Cu) (net 29))
+  (segment (start 151.15 111.77589) (end 151.15 106.7) (width 0.2) (layer F.Cu) (net 29))
+  (segment (start 151.765 112.39089) (end 151.15 111.77589) (width 0.2) (layer F.Cu) (net 29))
+  (segment (start 153.65 105.5) (end 153.65 102.85) (width 0.2) (layer F.Cu) (net 30))
+  (segment (start 153.65 102.85) (end 152.4 101.6) (width 0.2) (layer F.Cu) (net 30))
+  (segment (start 151.765 107.385) (end 153.65 105.5) (width 0.2) (layer F.Cu) (net 30))
+  (segment (start 151.765 111.12089) (end 151.765 107.385) (width 0.2) (layer F.Cu) (net 30))
+  (segment (start 152.4 108) (end 154.94 105.46) (width 0.2) (layer F.Cu) (net 31))
+  (segment (start 154.94 105.46) (end 154.94 104.14) (width 0.2) (layer F.Cu) (net 31))
+  (segment (start 152.4 111.75589) (end 152.4 108) (width 0.2) (layer F.Cu) (net 31))
+  (segment (start 153.035 112.39089) (end 152.4 111.75589) (width 0.2) (layer F.Cu) (net 31))
+  (segment (start 156.2 105.5) (end 156.2 102.86) (width 0.2) (layer F.Cu) (net 32))
+  (segment (start 156.2 102.86) (end 154.94 101.6) (width 0.2) (layer F.Cu) (net 32))
+  (segment (start 153.035 108.665) (end 156.2 105.5) (width 0.2) (layer F.Cu) (net 32))
+  (segment (start 153.035 111.12089) (end 153.035 108.665) (width 0.2) (layer F.Cu) (net 32))
+  (segment (start 153.65 109.35) (end 157.48 105.52) (width 0.2) (layer F.Cu) (net 33))
+  (segment (start 157.48 105.52) (end 157.48 104.14) (width 0.2) (layer F.Cu) (net 33))
+  (segment (start 153.65 111.75) (end 153.65 109.35) (width 0.2) (layer F.Cu) (net 33))
+  (segment (start 154.29089 112.39089) (end 153.65 111.75) (width 0.2) (layer F.Cu) (net 33))
+  (segment (start 154.305 112.39089) (end 154.29089 112.39089) (width 0.2) (layer F.Cu) (net 33))
+  (segment (start 158.75 105.45) (end 158.75 102.87) (width 0.2) (layer F.Cu) (net 34))
+  (segment (start 158.75 102.87) (end 157.48 101.6) (width 0.2) (layer F.Cu) (net 34))
+  (segment (start 154.305 109.895) (end 158.75 105.45) (width 0.2) (layer F.Cu) (net 34))
+  (segment (start 154.305 111.12089) (end 154.305 109.895) (width 0.2) (layer F.Cu) (net 34))
+  (segment (start 154.95 110.55) (end 160.02 105.48) (width 0.2) (layer F.Cu) (net 35))
+  (segment (start 160.02 105.48) (end 160.02 104.14) (width 0.2) (layer F.Cu) (net 35))
+  (segment (start 154.95 111.76589) (end 154.95 110.55) (width 0.2) (layer F.Cu) (net 35))
+  (segment (start 155.575 112.39089) (end 154.95 111.76589) (width 0.2) (layer F.Cu) (net 35))
+  (segment (start 161.3 104.9) (end 161.3 102.88) (width 0.2) (layer F.Cu) (net 36))
+  (segment (start 161.3 102.88) (end 160.02 101.6) (width 0.2) (layer F.Cu) (net 36))
+  (segment (start 155.575 110.625) (end 161.3 104.9) (width 0.2) (layer F.Cu) (net 36))
+  (segment (start 155.575 111.12089) (end 155.575 110.625) (width 0.2) (layer F.Cu) (net 36))
 )

Commit message: updated version number, silk screen spots
Parts:
- N2: value V20180610 -> V20180705
Changed lines of the file:
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@@
   (general
     (links 44)
-    (no_connects 32)
+    (no_connects 0)
     (area 127.924999 85.424999 172.075001 114.575001)
     (thickness 1.6)
@@
   )
   (setup
-    (last_trace_width 0.2)
+    (last_trace_width 0.127)
     (user_trace_width 0.127)
     (user_trace_width 0.2)
@@
       (effects (font (size 1 1) (thickness 0.15)))
     )
-    (fp_text value V20180610 (at -0.33 -0.455 90) (layer F.SilkS)
+    (fp_text value V20180705 (at -0.33 -0.455 90) (layer F.SilkS)
       (effects (font (size 1 1) (thickness 0.15)))
     )
@@
   (module SquantorConnectors:Header-0127-2X10-H006 locked (layer F.Cu)
     (at 149.86 88.265)
-    (fp_text reference J1 (at 0 -2.5) (layer F.SilkS)
+    (fp_text reference J1 (at 7.74 -0.065) (layer F.SilkS)
       (effects (font (size 1 1) (thickness 0.15)))
     )
@@
   (module SquantorConnectors:Header-0127-2X10-H006 locked (layer F.Cu)
     (at 149.86 111.76)
-    (fp_text reference J2 (at 0 -2.5) (layer F.SilkS)
+    (fp_text reference J2 (at -7.96 0.04) (layer F.SilkS)
       (effects (font (size 1 1) (thickness 0.15)))
     )
@@
     (tags "PIN HEADER")
     (attr virtual)
-    (fp_text reference J4 (at 0 -3.5) (layer F.SilkS)
+    (fp_text reference J4 (at -13.69 0.03) (layer F.SilkS)
       (effects (font (size 1 1) (thickness 0.15)))
     )
@@
     (tags "PIN HEADER")
     (attr virtual)
-    (fp_text reference J3 (at 0 -3.5) (layer F.SilkS)
-      (effects (font (size 1 1) (thickness 0.15)))
-    )
+    (fp_text reference J3 (at -13.79 0.01) (layer F.SilkS)
+      (effects (font (size 1 1) (thickness 0.15)))
+    )

Commit message: switched to two layer
Other:
- copper layers 4 -> 2
Changed lines of the file:
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@@
     (links 44)
     (no_connects 0)
-    (area 127.924999 85.424999 172.075001 114.575001)
+    (area 127.924999 84.348 173.002 115.752)
     (thickness 1.6)
     (drawings 10)
@@
   (layers
     (0 F.Cu signal)
-    (1 In1.Cu signal)
-    (2 In2.Cu signal)
     (31 B.Cu signal)
     (32 B.Adhes user)
