File: hardware/chrome_bee_lpc824/chrome_bee_lpc824.sch (KiCad schematic (older format))
At the start: 28 parts, among them J1 DevBoardDigital, J2 DevBoardAnalog, J3 JTAG_2X05, J4 POWER_IN, J5 BMP_UART, U1 POWER_JOINER, U2 POWER_JOINER, U3 MCP1702-MB, U4 POWER_JOINER, U5 LPC824M201JHI33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

Commit message: added updated lib references added vref
Parts:
- removed R7: 10, SquantorRcl:R_0402_hand, symbol Device:R
- added C?: 100n, SquantorRcl:C_0402, symbol Device:C
- added C?: 10mu, SquantorRcl:C_0805, symbol Device:C
- added U?: MCP1525, symbol SquantorMicrochip:MCP1525
Connections:
- net labels removed: IO14, IO15
- wire segments 126 -> 134
- no-connect marks 2 -> 5
Changed lines of the file:
@@
-$EndComp
-$Comp
-L Device:R R7
-U 1 1 5B861ACB
-P 10700 6000
-F 0 "R7" V 10907 6000 50  0000 C CNN
-F 1 "10" V 10816 6000 50  0000 C CNN
-F 2 "SquantorRcl:R_0402_hand" V 10630 6000 50  0001 C CNN
-F 3 "~" H 10700 6000 50  0001 C CNN
-	1    10700 6000
-	0    -1   -1   0
 $EndComp
 $Comp
@@
 L power:VDD #PWR0119
 U 1 1 5B862B4A
-P 10900 6000
-F 0 "#PWR0119" H 10900 5850 50  0001 C CNN
-F 1 "VDD" V 10918 6127 50  0000 L CNN
-F 2 "" H 10900 6000 50  0001 C CNN
-F 3 "" H 10900 6000 50  0001 C CNN
-	1    10900 6000
-	0    1    1    0
-$EndComp
-Wire Wire Line
-	10850 6000 10900 6000
+P 10550 6000
+F 0 "#PWR0119" H 10550 5850 50  0001 C CNN
+F 1 "VDD" V 10568 6127 50  0000 L CNN
+F 2 "" H 10550 6000 50  0001 C CNN
+F 3 "" H 10550 6000 50  0001 C CNN
+	1    10550 6000
+	0    1    1    0
+$EndComp
 Wire Wire Line
 	10600 6400 10550 6400
@@
 	2100 1800 2150 1800
 Wire Wire Line
-	2100 1900 2150 1900
-Wire Wire Line
 	1000 1400 950  1400
 Wire Wire Line
@@
 Wire Wire Line
 	1000 1800 950  1800
-Wire Wire Line
-	1000 1900 950  1900
 Text Label 2150 1300 0    50   ~ 0
 IO02_MOSI
@@
 Text Label 950  1800 2    50   ~ 0
 IO13
-Text Label 2150 1900 0    50   ~ 0
-IO14
-Text Label 950  1900 2    50   ~ 0
-IO15
 $Comp
 L SquantorNxp:LPC824M201JHI33 U5
@@
 	0    1    1    0
 $EndComp
-$Comp
-L power:VCC #PWR0146
-U 1 1 5BBC461A
-P 1650 4350
-F 0 "#PWR0146" H 1650 4200 50  0001 C CNN
-F 1 "VCC" H 1667 4523 50  0000 C CNN
-F 2 "" H 1650 4350 50  0001 C CNN
-F 3 "" H 1650 4350 50  0001 C CNN
-	1    1650 4350
-	0    1    1    0
-$EndComp
 Text Label 1900 4550 0    50   ~ 0
 IO06_TXO
@@
 Wire Wire Line
 	9900 2650 9850 2650
+$Comp
+L power:VDD #PWR0146
+U 1 1 5BC23CB9
+P 1650 4350
+F 0 "#PWR0146" H 1650 4200 50  0001 C CNN
+F 1 "VDD" V 1668 4477 50  0000 L CNN
+F 2 "" H 1650 4350 50  0001 C CNN
+F 3 "" H 1650 4350 50  0001 C CNN
+	1    1650 4350
+	0    1    1    0
+$EndComp
+NoConn ~ 2100 1900
+NoConn ~ 1000 1900
+NoConn ~ 1950 2750
+$Comp
+L SquantorMicrochip:MCP1525 U?
+U 1 1 5BC23232
+P 7600 4050
+F 0 "U?" H 7600 4300 60  0000 C CNN
+F 1 "MCP1525" H 7950 3900 60  0000 C CNN
+F 2 "" H 7600 4050 60  0001 C CNN
+F 3 "" H 7600 4050 60  0001 C CNN
+	1    7600 4050
+	1    0    0    -1
+$EndComp
+$Comp
+L power:VSSA #PWR?
+U 1 1 5BC2345A
+P 7850 4050
+F 0 "#PWR?" H 7850 3900 50  0001 C CNN
+F 1 "VSSA" V 7868 4177 50  0000 L CNN
+F 2 "" H 7850 4050 50  0001 C CNN
+F 3 "" H 7850 4050 50  0001 C CNN
+	1    7850 4050
+	0    1    1    0
+$EndComp
+Wire Wire Line
+	7300 4150 7350 4150
+Text Label 7300 4150 2    50   ~ 0
+VREF
+$Comp
+L power:VDDA #PWR?
+U 1 1 5BC303E7
+P 7300 3950
+F 0 "#PWR?" H 7300 3800 50  0001 C CNN
+F 1 "VDDA" V 7318 4078 50  0000 L CNN
+F 2 "" H 7300 3950 50  0001 C CNN
+F 3 "" H 7300 3950 50  0001 C CNN
+	1    7300 3950
+	0    -1   -1   0
+$EndComp
+Wire Wire Line
+	7400 3950 7350 3950
+Wire Wire Line
+	7850 4050 7800 4050
+$Comp
+L power:VSSA #PWR?
+U 1 1 5BC3D938
+P 7850 3650
+F 0 "#PWR?" H 7850 3500 50  0001 C CNN
+F 1 "VSSA" V 7868 3777 50  0000 L CNN
+F 2 "" H 7850 3650 50  0001 C CNN
+F 3 "" H 7850 3650 50  0001 C CNN
+	1    7850 3650
+	0    1    1    0
+$EndComp
+$Comp
+L Device:C C?
+U 1 1 5BC442D5
+P 7600 3650
+F 0 "C?" H 7715 3696 50  0000 L CNN
+F 1 "100n" H 7715 3605 50  0000 L CNN
+F 2 "SquantorRcl:C_0402" H 7638 3500 50  0001 C CNN
+F 3 "~" H 7600 3650 50  0001 C CNN
+	1    7600 3650
+	0    -1   -1   0
+$EndComp
+Wire Wire Line
+	7850 3650 7750 3650
+$Comp
+L power:VSSA #PWR?
+U 1 1 5BC51AB4
+P 7850 4400
+F 0 "#PWR?" H 7850 4250 50  0001 C CNN
+F 1 "VSSA" V 7868 4527 50  0000 L CNN
+F 2 "" H 7850 4400 50  0001 C CNN
+F 3 "" H 7850 4400 50  0001 C CNN
+	1    7850 4400
+	0    1    1    0
+$EndComp
+Wire Wire Line
+	7850 4400 7750 4400
+Wire Wire Line
+	7450 4400 7350 4400
+Wire Wire Line
+	7350 4400 7350 4150
+Connection ~ 7350 4150
+Wire Wire Line
+	7350 4150 7400 4150
+Wire Wire Line
+	7350 3950 7350 3650
+Wire Wire Line
+	7350 3650 7450 3650
+Connection ~ 7350 3950
+Wire Wire Line
+	7350 3950 7300 3950
+$Comp
+L Device:C C?
+U 1 1 5BC66DF6
+P 7600 4400
+F 0 "C?" H 7715 4446 50  0000 L CNN
+F 1 "10mu" H 7715 4355 50  0000 L CNN
+F 2 "SquantorRcl:C_0805" H 7638 4250 50  0001 C CNN
+F 3 "~" H 7600 4400 50  0001 C CNN
+	1    7600 4400
+	0    1    1    0
+$EndComp
 $EndSCHEMATC

Commit message: updated pcbcomponent library updated project with proper power joiners
Parts:
- U1, U2, U4: footprint SquantorRcl:R_0402_hand -> SquantorSpecial:power_joiner_05mm
- U6: renamed from U?; footprint (none) -> SquantorIC:SOT23-3-Microchip-TT
- gave numbers to parts that had none: 2
Changed lines of the file:
@@
 F 0 "U2" H 7450 5637 60  0000 C CNN
 F 1 "POWER_JOINER" H 7450 5531 60  0000 C CNN
-F 2 "SquantorRcl:R_0402_hand" H 7450 5350 60  0001 C CNN
+F 2 "SquantorSpecial:power_joiner_05mm" H 7450 5350 60  0001 C CNN
 F 3 "" H 7450 5350 60  0001 C CNN
 	1    7450 5350
@@
 F 0 "U1" H 7450 5187 60  0000 C CNN
 F 1 "POWER_JOINER" H 7450 5081 60  0000 C CNN
-F 2 "SquantorRcl:R_0402_hand" H 7450 4900 60  0001 C CNN
+F 2 "SquantorSpecial:power_joiner_05mm" H 7450 4900 60  0001 C CNN
 F 3 "" H 7450 4900 60  0001 C CNN
 	1    7450 4900
@@
 F 0 "U4" H 9200 4850 60  0000 C CNN
 F 1 "POWER_JOINER" H 9400 4550 60  0000 C CNN
-F 2 "SquantorRcl:R_0402_hand" H 9200 4700 60  0001 C CNN
+F 2 "SquantorSpecial:power_joiner_05mm" H 9200 4700 60  0001 C CNN
 F 3 "" H 9200 4700 60  0001 C CNN
 	1    9200 4700
@@
 NoConn ~ 1950 2750
 $Comp
-L SquantorMicrochip:MCP1525 U?
+L SquantorMicrochip:MCP1525 U6
 U 1 1 5BC23232
 P 7600 4050
-F 0 "U?" H 7600 4300 60  0000 C CNN
+F 0 "U6" H 7600 4300 60  0000 C CNN
 F 1 "MCP1525" H 7950 3900 60  0000 C CNN
-F 2 "" H 7600 4050 60  0001 C CNN
+F 2 "SquantorIC:SOT23-3-Microchip-TT" H 7600 4050 60  0001 C CNN
 F 3 "" H 7600 4050 60  0001 C CNN
 	1    7600 4050
@@
 $EndComp
 $Comp
-L power:VSSA #PWR?
+L power:VSSA #PWR0147
 U 1 1 5BC2345A
 P 7850 4050
-F 0 "#PWR?" H 7850 3900 50  0001 C CNN
+F 0 "#PWR0147" H 7850 3900 50  0001 C CNN
 F 1 "VSSA" V 7868 4177 50  0000 L CNN
 F 2 "" H 7850 4050 50  0001 C CNN
@@
 VREF
 $Comp
-L power:VDDA #PWR?
+L power:VDDA #PWR0148
 U 1 1 5BC303E7
 P 7300 3950
-F 0 "#PWR?" H 7300 3800 50  0001 C CNN
+F 0 "#PWR0148" H 7300 3800 50  0001 C CNN
 F 1 "VDDA" V 7318 4078 50  0000 L CNN
 F 2 "" H 7300 3950 50  0001 C CNN
@@
 	7850 4050 7800 4050
 $Comp
-L power:VSSA #PWR?
+L power:VSSA #PWR0149
 U 1 1 5BC3D938
 P 7850 3650
-F 0 "#PWR?" H 7850 3500 50  0001 C CNN
+F 0 "#PWR0149" H 7850 3500 50  0001 C CNN
 F 1 "VSSA" V 7868 3777 50  0000 L CNN
 F 2 "" H 7850 3650 50  0001 C CNN
@@
 $EndComp
 $Comp
-L Device:C C?
+L Device:C C7
 U 1 1 5BC442D5
 P 7600 3650
-F 0 "C?" H 7715 3696 50  0000 L CNN
+F 0 "C7" H 7715 3696 50  0000 L CNN
 F 1 "100n" H 7715 3605 50  0000 L CNN
 F 2 "SquantorRcl:C_0402" H 7638 3500 50  0001 C CNN
@@
 	7850 3650 7750 3650
 $Comp
-L power:VSSA #PWR?
+L power:VSSA #PWR0150
 U 1 1 5BC51AB4
 P 7850 4400
-F 0 "#PWR?" H 7850 4250 50  0001 C CNN
+F 0 "#PWR0150" H 7850 4250 50  0001 C CNN
 F 1 "VSSA" V 7868 4527 50  0000 L CNN
 F 2 "" H 7850 4400 50  0001 C CNN
@@
 	7350 3950 7300 3950
 $Comp
-L Device:C C?
+L Device:C C8
 U 1 1 5BC66DF6
 P 7600 4400
-F 0 "C?" H 7715 4446 50  0000 L CNN
+F 0 "C8" H 7715 4446 50  0000 L CNN
 F 1 "10mu" H 7715 4355 50  0000 L CNN
 F 2 "SquantorRcl:C_0805" H 7638 4250 50  0001 C CNN

Commit message: added _autosave to gitignores updated chrome bee project while messing about with net ties changed the symbol and footprint tables
Parts:
- removed U1, U2, U4: POWER_JOINER, SquantorSpecial:power_joiner_05mm, symbol SquantorRCL:POWER_JOINER
- added U1, U2, U4: POWER_JOINER, SquantorSpecial:power_joiner_05mm, symbol SquantorSpecial:POWER_JOINER
Changed lines of the file:
@@
-$EndComp
-$Comp
-L SquantorRCL:POWER_JOINER U2
-U 1 1 5BC8182D
-P 7450 5350
-F 0 "U2" H 7450 5637 60  0000 C CNN
-F 1 "POWER_JOINER" H 7450 5531 60  0000 C CNN
-F 2 "SquantorSpecial:power_joiner_05mm" H 7450 5350 60  0001 C CNN
-F 3 "" H 7450 5350 60  0001 C CNN
-	1    7450 5350
-	1    0    0    -1
-$EndComp
-$Comp
-L SquantorRCL:POWER_JOINER U1
-U 1 1 5BC819B4
-P 7450 4900
-F 0 "U1" H 7450 5187 60  0000 C CNN
-F 1 "POWER_JOINER" H 7450 5081 60  0000 C CNN
-F 2 "SquantorSpecial:power_joiner_05mm" H 7450 4900 60  0001 C CNN
-F 3 "" H 7450 4900 60  0001 C CNN
-	1    7450 4900
-	1    0    0    -1
 $EndComp
 $Comp
@@
 $EndComp
 $Comp
-L SquantorRCL:POWER_JOINER U4
-U 1 1 5BC9D12F
-P 9200 4700
-F 0 "U4" H 9200 4850 60  0000 C CNN
-F 1 "POWER_JOINER" H 9400 4550 60  0000 C CNN
-F 2 "SquantorSpecial:power_joiner_05mm" H 9200 4700 60  0001 C CNN
-F 3 "" H 9200 4700 60  0001 C CNN
-	1    9200 4700
-	1    0    0    -1
-$EndComp
-$Comp
 L power:VDD #PWR0138
 U 1 1 5BC9D294
@@
 	0    1    1    0
 $EndComp
+$Comp
+L SquantorSpecial:POWER_JOINER U1
+U 1 1 5BC3440E
+P 7450 4900
+F 0 "U1" H 7450 5187 60  0000 C CNN
+F 1 "POWER_JOINER" H 7450 5081 60  0000 C CNN
+F 2 "SquantorSpecial:power_joiner_05mm" H 7450 4900 60  0001 C CNN
+F 3 "" H 7450 4900 60  0001 C CNN
+	1    7450 4900
+	1    0    0    -1
+$EndComp
+$Comp
+L SquantorSpecial:POWER_JOINER U2
+U 1 1 5BC34537
+P 7450 5350
+F 0 "U2" H 7450 5637 60  0000 C CNN
+F 1 "POWER_JOINER" H 7450 5531 60  0000 C CNN
+F 2 "SquantorSpecial:power_joiner_05mm" H 7450 5350 60  0001 C CNN
+F 3 "" H 7450 5350 60  0001 C CNN
+	1    7450 5350
+	1    0    0    -1
+$EndComp
+$Comp
+L SquantorSpecial:POWER_JOINER U4
+U 1 1 5BC34597
+P 9200 4700
+F 0 "U4" H 9200 4987 60  0000 C CNN
+F 1 "POWER_JOINER" H 9200 4881 60  0000 C CNN
+F 2 "SquantorSpecial:power_joiner_05mm" H 9200 4700 60  0001 C CNN
+F 3 "" H 9200 4700 60  0001 C CNN
+	1    9200 4700
+	1    0    0    -1
+$EndComp
 $EndSCHEMATC

Commit message: updated chrome bee devboard
Parts:
- removed U1, U2, U4: POWER_JOINER, SquantorSpecial:power_joiner_05mm, symbol SquantorSpecial:POWER_JOINER
- added NT1, NT2, NT3: Net-Tie_2, SquantorSpecial:NetTie-2_SMD_Pad0.4mm, symbol Device:Net-Tie_2
Connections:
- wire segments 134 -> 143
Changed lines of the file:
@@
 L power:GND #PWR0132
 U 1 1 5BC86E20
-P 7150 4900
-F 0 "#PWR0132" H 7150 4650 50  0001 C CNN
-F 1 "GND" V 7155 4772 50  0000 R CNN
-F 2 "" H 7150 4900 50  0001 C CNN
-F 3 "" H 7150 4900 50  0001 C CNN
-	1    7150 4900
+P 7500 4950
+F 0 "#PWR0132" H 7500 4700 50  0001 C CNN
+F 1 "GND" V 7505 4822 50  0000 R CNN
+F 2 "" H 7500 4950 50  0001 C CNN
+F 3 "" H 7500 4950 50  0001 C CNN
+	1    7500 4950
 	0    1    1    0
 $EndComp
@@
 L power:GND #PWR0133
 U 1 1 5BC86EFB
-P 7150 5350
-F 0 "#PWR0133" H 7150 5100 50  0001 C CNN
-F 1 "GND" V 7155 5222 50  0000 R CNN
-F 2 "" H 7150 5350 50  0001 C CNN
-F 3 "" H 7150 5350 50  0001 C CNN
-	1    7150 5350
+P 7500 5400
+F 0 "#PWR0133" H 7500 5150 50  0001 C CNN
+F 1 "GND" V 7505 5272 50  0000 R CNN
+F 2 "" H 7500 5400 50  0001 C CNN
+F 3 "" H 7500 5400 50  0001 C CNN
+	1    7500 5400
 	0    1    1    0
 $EndComp
@@
 L power:VSS #PWR0134
 U 1 1 5BC8708C
-P 7750 4900
-F 0 "#PWR0134" H 7750 4750 50  0001 C CNN
-F 1 "VSS" V 7768 5028 50  0000 L CNN
-F 2 "" H 7750 4900 50  0001 C CNN
-F 3 "" H 7750 4900 50  0001 C CNN
-	1    7750 4900
+P 7850 4950
+F 0 "#PWR0134" H 7850 4800 50  0001 C CNN
+F 1 "VSS" V 7868 5078 50  0000 L CNN
+F 2 "" H 7850 4950 50  0001 C CNN
+F 3 "" H 7850 4950 50  0001 C CNN
+	1    7850 4950
 	0    1    1    0
 $EndComp
@@
 L power:VSSA #PWR0135
 U 1 1 5BC870FF
-P 7750 5350
-F 0 "#PWR0135" H 7750 5200 50  0001 C CNN
-F 1 "VSSA" V 7768 5477 50  0000 L CNN
-F 2 "" H 7750 5350 50  0001 C CNN
-F 3 "" H 7750 5350 50  0001 C CNN
-	1    7750 5350
-	0    1    1    0
-$EndComp
-Wire Wire Line
-	7150 4900 7200 4900
-Wire Wire Line
-	7150 5350 7200 5350
-Wire Wire Line
-	7700 4900 7750 4900
-Wire Wire Line
-	7750 5350 7700 5350
+P 7850 5400
+F 0 "#PWR0135" H 7850 5250 50  0001 C CNN
+F 1 "VSSA" V 7868 5527 50  0000 L CNN
+F 2 "" H 7850 5400 50  0001 C CNN
+F 3 "" H 7850 5400 50  0001 C CNN
+	1    7850 5400
+	0    1    1    0
+$EndComp
+Wire Wire Line
+	7500 4950 7550 4950
+Wire Wire Line
+	7500 5400 7550 5400
+Wire Wire Line
+	7850 5400 7800 5400
 $Comp
 L power:GND #PWR0136
@@
 L power:VDDA #PWR0139
 U 1 1 5BC9D326
-P 9500 4700
-F 0 "#PWR0139" H 9500 4550 50  0001 C CNN
-F 1 "VDDA" V 9518 4828 50  0000 L CNN
-F 2 "" H 9500 4700 50  0001 C CNN
-F 3 "" H 9500 4700 50  0001 C CNN
-	1    9500 4700
+P 9250 4700
+F 0 "#PWR0139" H 9250 4550 50  0001 C CNN
+F 1 "VDDA" V 9268 4828 50  0000 L CNN
+F 2 "" H 9250 4700 50  0001 C CNN
+F 3 "" H 9250 4700 50  0001 C CNN
+	1    9250 4700
 	0    1    1    0
 $EndComp
@@
 	8900 4700 8900 4650
 Wire Wire Line
-	9450 4700 9500 4700
+	9150 4700 9200 4700
 $Comp
 L power:VCC #PWR0140
@@
 $EndComp
 $Comp
-L SquantorSpecial:POWER_JOINER U1
-U 1 1 5BC3440E
-P 7450 4900
-F 0 "U1" H 7450 5187 60  0000 C CNN
-F 1 "POWER_JOINER" H 7450 5081 60  0000 C CNN
-F 2 "SquantorSpecial:power_joiner_05mm" H 7450 4900 60  0001 C CNN
-F 3 "" H 7450 4900 60  0001 C CNN
-	1    7450 4900
-	1    0    0    -1
-$EndComp
-$Comp
-L SquantorSpecial:POWER_JOINER U2
-U 1 1 5BC34537
-P 7450 5350
-F 0 "U2" H 7450 5637 60  0000 C CNN
-F 1 "POWER_JOINER" H 7450 5531 60  0000 C CNN
-F 2 "SquantorSpecial:power_joiner_05mm" H 7450 5350 60  0001 C CNN
-F 3 "" H 7450 5350 60  0001 C CNN
-	1    7450 5350
-	1    0    0    -1
-$EndComp
-$Comp
-L SquantorSpecial:POWER_JOINER U4
-U 1 1 5BC34597
-P 9200 4700
-F 0 "U4" H 9200 4987 60  0000 C CNN
-F 1 "POWER_JOINER" H 9200 4881 60  0000 C CNN
-F 2 "SquantorSpecial:power_joiner_05mm" H 9200 4700 60  0001 C CNN
-F 3 "" H 9200 4700 60  0001 C CNN
-	1    9200 4700
-	1    0    0    -1
-$EndComp
+L Device:Net-Tie_2 NT1
+U 1 1 5BC25B05
+P 7650 4950
+F 0 "NT1" H 7650 5128 50  0000 C CNN
+F 1 "Net-Tie_2" H 7650 5037 50  0000 C CNN
+F 2 "SquantorSpecial:NetTie-2_SMD_Pad0.4mm" H 7650 4950 50  0001 C CNN
+F 3 "~" H 7650 4950 50  0001 C CNN
+	1    7650 4950
+	1    0    0    -1
+$EndComp
+$Comp
+L Device:Net-Tie_2 NT2
+U 1 1 5BC25BA5
+P 7650 5400
+F 0 "NT2" H 7650 5578 50  0000 C CNN
+F 1 "Net-Tie_2" H 7650 5487 50  0000 C CNN
+F 2 "SquantorSpecial:NetTie-2_SMD_Pad0.4mm" H 7650 5400 50  0001 C CNN
+F 3 "~" H 7650 5400 50  0001 C CNN
+	1    7650 5400
+	1    0    0    -1
+$EndComp
+$Comp
+L Device:Net-Tie_2 NT3
+U 1 1 5BC25C46
+P 9050 4700
+F 0 "NT3" H 9050 4878 50  0000 C CNN
+F 1 "Net-Tie_2" H 9050 4787 50  0000 C CNN
+F 2 "SquantorSpecial:NetTie-2_SMD_Pad0.4mm" H 9050 4700 50  0001 C CNN
+F 3 "~" H 9050 4700 50  0001 C CNN
+	1    9050 4700
+	1    0    0    -1
+$EndComp
+$Comp
+L power:PWR_FLAG #FLG0102
+U 1 1 5BCB3101
+P 7850 5100
+F 0 "#FLG0102" H 7850 5175 50  0001 C CNN
+F 1 "PWR_FLAG" V 7850 5228 50  0000 L CNN
+F 2 "" H 7850 5100 50  0001 C CNN
+F 3 "~" H 7850 5100 50  0001 C CNN
+	1    7850 5100
+	0    1    1    0
+$EndComp
+Wire Wire Line
+	7850 5100 7800 5100
+Wire Wire Line
+	7800 5100 7800 4950
+Wire Wire Line
+	7750 4950 7800 4950
+Connection ~ 7800 4950
+Wire Wire Line
+	7800 4950 7850 4950
+$Comp
+L power:PWR_FLAG #FLG0101
+U 1 1 5BCC253A
+P 7850 5550
+F 0 "#FLG0101" H 7850 5625 50  0001 C CNN
+F 1 "PWR_FLAG" V 7850 5678 50  0000 L CNN
+F 2 "" H 7850 5550 50  0001 C CNN
+F 3 "~" H 7850 5550 50  0001 C CNN
+	1    7850 5550
+	0    1    1    0
+$EndComp
+Wire Wire Line
+	7850 5550 7800 5550
+Wire Wire Line
+	7800 5550 7800 5400
+Connection ~ 7800 5400
+Wire Wire Line
+	7800 5400 7750 5400
+$Comp
+L power:PWR_FLAG #FLG0103
+U 1 1 5BCD1D8A
+P 9250 4850
+F 0 "#FLG0103" H 9250 4925 50  0001 C CNN
+F 1 "PWR_FLAG" V 9250 4978 50  0000 L CNN
+F 2 "" H 9250 4850 50  0001 C CNN
+F 3 "~" H 9250 4850 50  0001 C CNN
+	1    9250 4850
+	0    1    1    0
+$EndComp
+Wire Wire Line
+	9250 4850 9200 4850
+Wire Wire Line
+	9200 4850 9200 4700
+Connection ~ 9200 4700
+Wire Wire Line
+	9200 4700 9250 4700
 $EndSCHEMATC

Commit message: checked if everything ports over to a new install
Parts:
- J4: symbol SquantorConnectors:POWER_IN -> SquantorConnectors:POWER_IN_2PIN
Changed lines of the file:
@@
 	9800 1200 9750 1200
 $Comp
-L SquantorConnectors:POWER_IN J4
+L SquantorConnectors:POWER_IN_2PIN J4
 U 1 1 5BC56C4A
 P 1350 3750

Commit message: further schematic extensions started layout
Parts:
- removed NT2: Net-Tie_2, SquantorSpecial:NetTie-2_SMD_Pad0.4mm, symbol Device:Net-Tie_2
- added R10, R9: 2.2k, SquantorRcl:R_0402_hand, symbol Device:R
- added R7, R8: 100, SquantorRcl:R_0402_hand, symbol Device:R
Connections:
- net VSSA is gone; now on net VSS: C4.2, C7.2, C8.1, J2.7 (VSSA), J2.8 (VSSA), U5.20 (VREFN), U6.3 (GND)
- net IO00_SDA: now also R10.1
- net IO01_SCL: now also R9.1
- net IO05_RXI: now also R7.2; no longer J5.2 (TXDO)
- net IO06_TXO: now also R8.2; no longer J5.3 (RXDI)
- net VDD: now also R10.2, R9.2
- new net: J5.2 (TXDO), R7.1
- new net: J5.3 (RXDI), R8.1
Other:
- moved on the sheet: C3, C4, C5, C6, C7, C8, NT1, NT3, U3, U6

Commit message: updates to chrome bee devboard
Parts:
- removed NT1, NT3: Net-Tie_2, SquantorSpecial:NetTie-2_SMD_Pad0.4mm, symbol Device:Net-Tie_2
- added C10: 1u, SquantorRcl:C_0603, symbol Device:C
- added C9: 100n, SquantorRcl:C_0402, symbol Device:C
- added FB1, FB2, FB3: Ferrite_Bead_Small, SquantorRcl:R_0402_hand, symbol Device:Ferrite_Bead_Small
- C3: value 100n -> 1u; footprint SquantorRcl:C_0402 -> SquantorRcl:C_0603
- C5: footprint SquantorRcl:C_0805 -> SquantorRcl:C_0603
- J3: footprint SquantorConnectors:Header-0127-2X05-SMD -> SquantorConnectors:Header-0127-2X05-H006
- J4: footprint Connectors_Molex:Molex_PicoBlade_53047-0210_02x1.25mm_Straight -> Connector_JST:JST_PH_S2B-PH-K_1x02_P2.00mm_Horizontal
- J5: footprint Connectors_Molex:Molex_PicoBlade_53047-0410_04x1.25mm_Straight -> Connector_JST:JST_PH_S4B-PH-K_1x04_P2.00mm_Horizontal
- N2: value 20180819 -> 20190121
Connections:
- net GND is gone; now on net VSS: C5.2, C6.2, J4.2 (GND), U3.1 (GND)
- net VDD: now also C7.1, J2.5 (VDDA), J2.6 (VDDA), U6.1 (VIN), FB1.2, FB2.2; no longer C3.1, U5.19 (VDD)
- net VSS: now also C9.2, FB3.2; no longer C4.2, U5.20 (VREFN)
- removed net VDDA: C4.1, C7.1, J2.5 (VDDA), J2.6 (VDDA), U5.21 (VREFP), U6.1 (VIN)
- new net: C3.1, C9.1, FB1.1, U5.19 (VDD)
- new net: C10.2, C4.2, FB3.1, U5.20 (VREFN)
- new net: C10.1, C4.1, FB2.1, U5.21 (VREFP)
Other:
- moved on the sheet: C5, C6, C7, C8, R10, R9, U3, U5A, U6
