File: hardware/hammond_1551G_devboard_Lipo_charger/hammond_1551G_devboard_Lipo_charger.sch (KiCad schematic (older format))
At the start: 25 parts, among them J1 DevBoardDigital, J2 DevBoardAnalog, J3 Battery_2pin, J4 DevBoardUartInput, J5 JTAG_2X05, Q1 Q_NMOS_GSD, U1 MCP1702-MB, U2 power_joiner_2_nets, U3 power_joiner_2_nets, U4 power_joiner_2_nets, U5 power_joiner_2_nets, U6 MCP738312-OT

Commit message: completed layout, time for silk screen updates
Connections:
- net GND: no longer J5.1 (VCC), J5.3 (GND), J5.5 (GND), J5.9 (GNDDET)
- net VSS: now also J5.1 (VCC), J5.3 (GND), J5.5 (GND), J5.9 (GNDDET)
- net VREG: now reaches C1.2, D1.1 (K), Q1.2 (S), U1.2 (Vin), U1.TAB (Vin)
Changed lines of the file:
@@
 P 4650 5150
 F 0 "U1" V 4950 5100 60  0000 R CNN
-F 1 "MCP1702-MB" V 5100 5450 60  0000 R CNN
+F 1 "MCP1702-MB" V 5100 5500 60  0000 R CNN
 F 2 "SquantorIC:SOT89-ViaTab-Microchip-MB" H 4650 5150 60  0001 C CNN
 F 3 "" H 4650 5150 60  0001 C CNN
@@
 F 3 "" H 1450 5250 60  0001 C CNN
 	1    1450 5100
-	1    0    0    -1
-$EndComp
-$Comp
-L power:GND #PWR0123
-U 1 1 5C4CBC11
-P 2000 5350
-F 0 "#PWR0123" H 2000 5100 50  0001 C CNN
-F 1 "GND" H 2005 5177 50  0000 C CNN
-F 2 "" H 2000 5350 50  0001 C CNN
-F 3 "" H 2000 5350 50  0001 C CNN
-	1    2000 5350
 	1    0    0    -1
 $EndComp
@@
 Wire Wire Line
 	5050 3950 5000 3950
+$Comp
+L power:VSS #PWR0123
+U 1 1 5C4DEF61
+P 2000 5350
+F 0 "#PWR0123" H 2000 5200 50  0001 C CNN
+F 1 "VSS" V 2017 5478 50  0000 L CNN
+F 2 "" H 2000 5350 50  0001 C CNN
+F 3 "" H 2000 5350 50  0001 C CNN
+	1    2000 5350
+	-1   0    0    1
+$EndComp
+Text Label 4400 4800 0    50   ~ 0
+VREG
 $EndSCHEMATC

Commit message: replaced JST PH connectors by SMD variants so they stack better, needed to redo layout altough :(
Parts:
- J3: footprint Connector_JST:JST_PH_S2B-PH-K_1x02_P2.00mm_Horizontal -> Connector_JST:JST_PH_S2B-PH-SM4-TB_1x02-1MP_P2.00mm_Horizontal
- J4: footprint Connector_JST:JST_PH_S4B-PH-K_1x04_P2.00mm_Horizontal -> Connector_JST:JST_PH_S4B-PH-SM4-TB_1x04-1MP_P2.00mm_Horizontal
Changed lines of the file:
@@
 F 0 "J3" H 1131 3646 50  0000 R CNN
 F 1 "Battery_2pin" H 1131 3555 50  0000 R CNN
-F 2 "Connector_JST:JST_PH_S2B-PH-K_1x02_P2.00mm_Horizontal" H 1550 3600 50  0001 C CNN
+F 2 "Connector_JST:JST_PH_S2B-PH-SM4-TB_1x02-1MP_P2.00mm_Horizontal" H 1550 3600 50  0001 C CNN
 F 3 "" H 1550 3600 50  0001 C CNN
 	1    1400 3600
@@
 F 0 "J4" H 1481 4715 50  0000 C CNN
 F 1 "DevBoardUartInput" H 1481 4624 50  0000 C CNN
-F 2 "Connector_JST:JST_PH_S4B-PH-K_1x04_P2.00mm_Horizontal" H 1450 4300 50  0001 C CNN
+F 2 "Connector_JST:JST_PH_S4B-PH-SM4-TB_1x04-1MP_P2.00mm_Horizontal" H 1450 4300 50  0001 C CNN
 F 3 "" H 1450 4300 50  0001 C CNN
 	1    1450 4300
