File: electronics/nuclone_RP2040/nuclone_RP2040.kicad_pcb (KiCad board)
At the start: 4 copper layers, 50 x 50 mm, 64 parts, among them J1 JTAG_2X05, J2 TYPE-C-31-M-12, J3 nuclone_small_left, J4 nuclone_small_right, J5 Conn_02x06_Odd_Even, SW1 RESET, SW2 Bootloader, U1 MCP1702-MB, U2 TPESD0504C6, U3 rp2040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

Commit message: further routing in progress
Parts:
- moved C12 7.49 mm to (87.4, 98.7), turned to -90 degrees
- moved C23 6.31 mm to (93.0, 81.9)
- moved C11 4.03 mm to (92.6, 98.7), turned to 90 degrees
- moved C4 2.16 mm to (98.2, 71.8), turned to -90 degrees
- moved R7 1.80 mm to (100.2, 71.3), turned to 180 degrees
- moved C7 1.27 mm to (86.2, 96.6)
- moved C15 1.27 mm to (87.3, 96.6)
- moved R9 1.27 mm to (85.1, 96.6)
- moved C16 1.15 mm to (85.0, 84.0)
- moved C21 1.15 mm to (83.9, 84.0)
- moved C8 1.15 mm to (86.1, 84.0)
- moved C13 1.04 mm to (91.3, 91.7)
- moved C10 0.60 mm to (90.8, 87.6)
- moved C19 0.45 mm to (90.2, 85.9)
- moved FB2 0.45 mm to (91.3, 85.9)
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Routing:
- net /GPIO_15: track 0.00 -> 37.2 mm
- net /GPIO_14: track 0.00 -> 33.4 mm
- net /GPIO_29: track 0.00 -> 23.7 mm
- net /GPIO_27: track 0.00 -> 22.3 mm
- net /GPIO_25: track 0.00 -> 21.3 mm
- net /GPIO_23: track 0.00 -> 20.6 mm
- net /GPIO_21: track 0.00 -> 20.6 mm
- net /GPIO_19: track 0.00 -> 19.8 mm
- net /GPIO_17: track 0.00 -> 19.8 mm
- net /GPIO_28: track 0.00 -> 18.9 mm
- net /GPIO_26: track 0.00 -> 17.5 mm
- net /GPIO_16: track 0.00 -> 16.8 mm
- net /GPIO_24: track 0.00 -> 16.8 mm
- net /GPIO_22: track 0.00 -> 16.1 mm
- net /GPIO_20: track 0.00 -> 16.0 mm
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
Commit message: more alignment to official schematic
Parts:
- added R10: DNF, SquantorRcl:R_0402_hand, F.Cu at (85.1, 80.5)
- added R11: 1K, SquantorRcl:R_0402_hand, F.Cu at (88.3, 80.5)
- N2: value V20220527 -> V20220707
- moved C13 0.40 mm to (91.7, 91.7)
- moved C21 0.20 mm to (83.7, 84.0)
- moved C16 0.10 mm to (84.9, 84.0)
Routing:
- net /VDD: track 36.0 -> 42.2 mm, vias 12 -> 15
- net /microcontroller/QSPI_SD1: track 10.7 -> 9.92 mm

Commit message: updated crystal, further placing and routing
Parts:
- Y1: footprint SquantorCrystal:Crystal_3225_4 -> SquantorCrystal:Crystal_2520_4
- moved C11 10.0 mm to (82.6, 99.2), turned to -90 degrees
- moved R11 6.53 mm to (82.2, 78.3), turned to -90 degrees
- moved Y1 5.12 mm to (84.9, 99.2), turned to 180 degrees
- moved R10 4.57 mm to (81.1, 78.3), turned to -90 degrees
- moved C12 0.54 mm to (87.2, 99.2), turned to 90 degrees
Routing:
- net Net-(C11-Pad2): track 0.00 -> 9.03 mm
- net /VSS: track 43.2 -> 50.5 mm, vias 29 -> 31
- net Net-(C12-Pad2): track 0.00 -> 3.39 mm
- net /GPIO_14: track 33.4 -> 34.0 mm
