File: electronics/nuclone_LPC804M101JHI33/microcontroller.kicad_sch (KiCad schematic)
At the start: 11 parts

Commit message: switched from testpins to debug connector
Parts:
- added J?: Conn_02x06_Odd_Even, SquantorConnectors:Header-0127-2X10-H006, symbol Connector_Generic:Conn_02x04_Odd_Even
- C3, C5, C6: value (none) -> 1u; footprint (none) -> SquantorRcl:C_0402
- C7, C8: value (none) -> 100n; footprint (none) -> SquantorRcl:C_0402
- FB2: value (none) -> 600; footprint (none) -> SquantorRcl:L_0402
- JP1: value (none) -> TMS/PIO0_2; footprint (none) -> SquantorSpecial:solder_jumper_0402_2way_noconn
- JP2: value (none) -> TCK/PIO0_3; footprint (none) -> SquantorSpecial:solder_jumper_0402_2way_noconn
- JP3: value (none) -> !RESET/PIO0_5; footprint (none) -> SquantorSpecial:solder_jumper_0402_2way_noconn
- JP4: value (none) -> VDDA; footprint (none) -> SquantorSpecial:solder_jumper_0402_2way_conn
- U3: value (none) -> LPC804M101JHI33; footprint (none) -> SquantorIC:SOT617-3_alt_paste
Connections:
- net RESET: now also J?.8 (Pin_8)
- net TCK: now also J?.6 (Pin_6)
- net TMS: now also J?.4 (Pin_4)
- net VSS: now also J?.1 (Pin_1), J?.3 (Pin_3), J?.5 (Pin_5), J?.7 (Pin_7)
- new net BOOTLOADER: J?.2 (Pin_2)
Other:
- note added: "QSPI debug connector"

Commit message: changed test points to a connector for logic analyser
Parts:
- J5: renamed from J?; footprint SquantorConnectors:Header-0127-2X10-H006 -> SquantorConnectors:Header-0127-2X04-H006
Connections:
- net BOOTLOADER is gone; now on net RESET: J5.2 (Pin_2)
- net RESET: no longer J5.8 (Pin_8)
- net TCK: now also J5.4 (Pin_4); no longer J5.6 (Pin_6)
- net TMS: now also J5.6 (Pin_6); no longer J5.4 (Pin_4)
- new net BOOT: J5.8 (Pin_8)
Changed lines of the file:
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@@
+    (stroke (width 0) (type default) (color 0 0 0 0))
+  )
+  (wire (pts (xy 24.13 50.8) (xy 25.4 50.8))
     (stroke (width 0) (type default) (color 0 0 0 0))
   )
@@
     (effects (font (size 1.27 1.27)) (justify right bottom))
   )
-  (label "TMS" (at 198.12 149.86 0)
+  (label "TMS" (at 198.12 152.4 0)
     (effects (font (size 1.27 1.27)) (justify left bottom))
   )
@@
     (effects (font (size 1.27 1.27)) (justify right bottom))
   )
-  (label "BOOTLOADER" (at 198.12 147.32 0)
+  (label "BOOTLOADER" (at 198.12 154.94 0)
     (effects (font (size 1.27 1.27)) (justify left bottom))
   )
@@
     (effects (font (size 1.27 1.27)) (justify right bottom))
   )
-  (label "TCK" (at 198.12 152.4 0)
+  (label "TCK" (at 198.12 149.86 0)
     (effects (font (size 1.27 1.27)) (justify left bottom))
   )
@@
     (effects (font (size 1.27 1.27)) (justify left bottom))
   )
+  (label "BOOTLOADER" (at 25.4 50.8 0)
+    (effects (font (size 1.27 1.27)) (justify left bottom))
+  )
   (label "PIO0_21" (at 242.57 74.93 180)
     (effects (font (size 1.27 1.27)) (justify right bottom))
@@
     (effects (font (size 1.27 1.27)) (justify right bottom))
   )
-  (label "RESET" (at 198.12 154.94 0)
+  (label "RESET" (at 198.12 147.32 0)
     (effects (font (size 1.27 1.27)) (justify left bottom))
   )
@@
   )
   (hierarchical_label "GPIO_23" (shape bidirectional) (at 24.13 111.76 180)
+    (effects (font (size 1.27 1.27)) (justify right))
+  )
+  (hierarchical_label "BOOT" (shape input) (at 24.13 50.8 180)
     (effects (font (size 1.27 1.27)) (justify right))
   )
@@
   (symbol (lib_id "Connector_Generic:Conn_02x04_Odd_Even") (at 189.23 149.86 0) (unit 1)
     (in_bom yes) (on_board yes)
-    (property "Reference" "J?" (id 0) (at 189.23 144.78 0))
+    (property "Reference" "J5" (id 0) (at 189.23 144.78 0))
     (property "Value" "Conn_02x06_Odd_Even" (id 1) (at 190.5 157.48 0))
-    (property "Footprint" "SquantorConnectors:Header-0127-2X10-H006" (id 2) (at 189.23 149.86 0)
-      (effects (font (size 1.27 1.27)) hide)
-    )
+    (property "Footprint" "SquantorConnectors:Header-0127-2X04-H006" (id 2) (at 189.23 149.86 0)
+      (effects (font (size 1.27 1.27)) hide)
+    )

Commit message: reviewed
Other:
- note added: "Testpads"
- note removed: "QSPI debug connector"
Changed lines of the file:
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@@
     (stroke (width 0) (type default) (color 0 0 0 0))
   )
-  (polyline (pts (xy 187.96 160.02) (xy 187.96 163.83))
+  (polyline (pts (xy 201.93 160.02) (xy 201.93 163.83))
     (stroke (width 0) (type default) (color 0 0 0 0))
   )
@@
     (stroke (width 0) (type default) (color 0 0 0 0))
   )
-  (polyline (pts (xy 212.09 160.02) (xy 187.96 160.02))
+  (polyline (pts (xy 212.09 160.02) (xy 201.93 160.02))
     (stroke (width 0) (type default) (color 0 0 0 0))
   )
@@
     (stroke (width 0) (type default) (color 0 0 0 0))
   )
-  (text "QSPI debug connector" (at 189.23 162.56 0)
+  (text "Testpads" (at 203.2 162.56 0)
     (effects (font (size 1.27 1.27)) (justify left bottom))
   )
