File: electronics/nuclone_RP2040_SON/microcontroller.kicad_sch (KiCad schematic)
At the start: 25 parts, among them J5 Conn_02x06_Odd_Even, U3 rp2040, U4 MX25L3233FZBI, Y1 12MHz

Commit message: ERC passes without errors, DRC without errors and warnings, updated versionnumber
Changed lines of the file:
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@@
+    (stroke (width 0) (type default) (color 0 0 0 0))
+  )
+  (wire (pts (xy 256.54 16.51) (xy 256.54 20.32))
     (stroke (width 0) (type default) (color 0 0 0 0))
   )
@@
   )
   (polyline (pts (xy 228.6 124.46) (xy 228.6 128.27))
+    (stroke (width 0) (type default) (color 0 0 0 0))
+  )
+  (wire (pts (xy 248.92 16.51) (xy 256.54 16.51))
     (stroke (width 0) (type default) (color 0 0 0 0))
   )
@@
     (pin "2")
   )
+  (symbol (lib_id "power:PWR_FLAG") (at 248.92 16.51 90) (unit 1)
+    (in_bom yes) (on_board yes) (fields_autoplaced)
+    (property "Reference" "#FLG0101" (id 0) (at 247.015 16.51 0)
+      (effects (font (size 1.27 1.27)) hide)
+    )
+    (property "Value" "PWR_FLAG" (id 1) (at 245.11 16.5099 90)
+      (effects (font (size 1.27 1.27)) (justify left))
+    )
+    (property "Footprint" "" (id 2) (at 248.92 16.51 0)
+      (effects (font (size 1.27 1.27)) hide)
+    )
+    (property "Datasheet" "~" (id 3) (at 248.92 16.51 0)
+      (effects (font (size 1.27 1.27)) hide)
+    )
+    (pin "1")
+  )
   (symbol (lib_id "Device:R") (at 226.06 99.06 90) (unit 1)
