File: electronics/nuclone_RP2040_SON/nuclone_RP2040_SON.kicad_sch (KiCad schematic)
At the start: 36 parts, among them J1 JTAG_2X05, J2 TYPE-C-31-M-12, J3 nuclone_small_left, J4 nuclone_small_right, SW1 RESET, SW2 Bootloader, U1 MCP1702-MB, U2 TPESD0504C6

Commit message: ERC passes without errors, DRC without errors and warnings, updated versionnumber
Parts:
- N2: value V20230129 -> V20230205
- N4: value NuClone RP2040 -> NuClone RP2040 SON
Connections:
- net Bootloader renamed BOOTLOADER
Changed lines of the file:
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@@
     (effects (font (size 1.27 1.27)) (justify left bottom))
   )
-  (label "Bootloader" (at 241.3 157.48 0)
+  (label "BOOTLOADER" (at 241.3 157.48 0)
     (effects (font (size 1.27 1.27)) (justify left bottom))
   )
@@
     (effects (font (size 1.27 1.27)) (justify right bottom))
   )
-  (label "Bootloader" (at 91.44 130.81 180)
+  (label "BOOTLOADER" (at 91.44 130.81 180)
     (effects (font (size 1.27 1.27)) (justify right bottom))
   )
@@
       (effects (font (size 1.524 1.524)) (justify left))
     )
-    (property "Value" "V20230129" (id 1) (at 17.78 182.88 0)
+    (property "Value" "V20230205" (id 1) (at 17.78 182.88 0)
       (effects (font (size 1.524 1.524)) (justify left))
     )
@@
       (effects (font (size 1.524 1.524)) (justify left))
     )
-    (property "Value" "NuClone RP2040" (id 1) (at 20.32 170.18 0)
+    (property "Value" "NuClone RP2040 SON" (id 1) (at 20.32 170.18 0)
       (effects (font (size 1.524 1.524)) (justify left))
     )
@@
       (reference "#FLG01") (unit 1) (value "PWR_FLAG") (footprint "")
     )
+    (path "/00000000-0000-0000-0000-00006127a958/a0817b32-ae2f-4edc-b714-ffc776c02071"
+      (reference "#FLG0101") (unit 1) (value "PWR_FLAG") (footprint "")
+    )
     (path "/00000000-0000-0000-0000-00005d820111"
       (reference "C1") (unit 1) (value "10u") (footprint "SquantorRcl:C_0603")
@@
     )
     (path "/00000000-0000-0000-0000-00005d6a68b9"
-      (reference "N2") (unit 1) (value "V20230129") (footprint "SquantorLabels:Label_Generic")
+      (reference "N2") (unit 1) (value "V20230205") (footprint "SquantorLabels:Label_Generic")
     )
     (path "/00000000-0000-0000-0000-00005d8b1b32"
@@
     )
     (path "/00000000-0000-0000-0000-00005fb0926c"
-      (reference "N4") (unit 1) (value "NuClone RP2040") (footprint "SquantorLabels:Label_Generic")
+      (reference "N4") (unit 1) (value "NuClone RP2040 SON") (footprint "SquantorLabels:Label_Generic")
     )
     (path "/00000000-0000-0000-0000-0000618b84bf"

Commit message: updated SON RP2040 nuclone
Parts:
- N2: value V20230205 -> V20230207
Changed lines of the file:
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@@
       (effects (font (size 1.524 1.524)) (justify left))
     )
-    (property "Value" "V20230205" (id 1) (at 17.78 182.88 0)
+    (property "Value" "V20230207" (id 1) (at 17.78 182.88 0)
       (effects (font (size 1.524 1.524)) (justify left))
     )
@@
     )
     (path "/00000000-0000-0000-0000-00005d6a68b9"
-      (reference "N2") (unit 1) (value "V20230205") (footprint "SquantorLabels:Label_Generic")
+      (reference "N2") (unit 1) (value "V20230207") (footprint "SquantorLabels:Label_Generic")
     )
     (path "/00000000-0000-0000-0000-00005d8b1b32"

Commit message: updated versionnumber
Parts:
- N2: value V20230207 -> V20230211
Changed lines of the file:
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@@
       (effects (font (size 1.524 1.524)) (justify left))
     )
-    (property "Value" "V20230207" (id 1) (at 17.78 182.88 0)
+    (property "Value" "V20230211" (id 1) (at 17.78 182.88 0)
       (effects (font (size 1.524 1.524)) (justify left))
     )
@@
     )
     (path "/00000000-0000-0000-0000-00005d6a68b9"
-      (reference "N2") (unit 1) (value "V20230207") (footprint "SquantorLabels:Label_Generic")
+      (reference "N2") (unit 1) (value "V20230211") (footprint "SquantorLabels:Label_Generic")
     )
     (path "/00000000-0000-0000-0000-00005d8b1b32"
