File: electronics/nuclone_LPC804M101DH24/microcontroller.kicad_sch (KiCad schematic)
At the start: 13 parts, among them J5 Conn_02x06_Odd_Even, U2 LPC804M101JHI33, U3 reference_sot23-3

Commit message: routed, silk placed, changed labels
Connections:
- net VDD: no longer C10.2
- net VREFP: now also C10.2; no longer C10.1
- net VSS: now also C10.1
Changed lines of the file:
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@@
     (effects (font (size 1.27 1.27)) (justify left bottom))
+  )
+  (label "VSS" (at 149.86 52.07 180) (fields_autoplaced)
+    (effects (font (size 1.27 1.27)) (justify right bottom))
   )
   (label "GPIO_11" (at 99.06 123.19 180) (fields_autoplaced)
@@
     (effects (font (size 1.27 1.27)) (justify left bottom))
   )
-  (label "VREFP" (at 149.86 52.07 180) (fields_autoplaced)
-    (effects (font (size 1.27 1.27)) (justify right bottom))
-  )
-  (label "VDD" (at 157.48 52.07 0) (fields_autoplaced)
-    (effects (font (size 1.27 1.27)) (justify left bottom))
-  )
+  (label "VREFP" (at 157.48 52.07 0) (fields_autoplaced)
+    (effects (font (size 1.27 1.27)) (justify left bottom))
+  )

Commit message: added crystal oscillator
Parts:
- added C11: 1u, SquantorCapacitor:C_0603, symbol Device:C
- added JP5: OSC to GPIO_01, SquantorSpecial:solder_jumper_0402_2way_noconn, symbol SquantorSpecial:Solderjumper_2way_noconn
- added R10, R11: 10K, SquantorResistor:R_0603_hand, symbol Device:R
- added U4: TBD, SquantorCrystal:Crystal_3225_4_hand, symbol SquantorGenericDigital:OSC_3state
Connections:
- net GPIO_23: now also JP5.2
- net VDD: now also C11.2, R11.2, U4.4 (VDD)
- net VSS: now also C11.1, R10.2, U4.2 (GND)
- new net OSC_EN: R10.1, R11.1, U4.1 (Tri)
- new net OSC_OUT: JP5.1, U4.3 (OUT)
Changed lines of the file:
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@@
+    (stroke (width 0) (type default))
+  )
+  (wire (pts (xy 146.05 72.39) (xy 149.86 72.39))
     (stroke (width 0) (type default))
   )
@@
     (stroke (width 0) (type default))
   )
+  (wire (pts (xy 146.05 74.93) (xy 146.05 72.39))
+    (stroke (width 0) (type default))
+  )
   (wire (pts (xy 24.13 33.02) (xy 25.4 33.02))
     (stroke (width 0) (type default))
@@
     (stroke (width 0) (type default))
   )
+  (wire (pts (xy 149.86 74.93) (xy 146.05 74.93))
+    (stroke (width 0) (type default))
+  )
   (wire (pts (xy 24.13 111.76) (xy 25.4 111.76))
     (stroke (width 0) (type default))
@@
     (effects (font (size 1.27 1.27)) (justify right bottom))
   )
+  (label "OSC_EN" (at 146.05 72.39 180) (fields_autoplaced)
+    (effects (font (size 1.27 1.27)) (justify right bottom))
+  )
   (label "VSS" (at 160.02 41.91 0) (fields_autoplaced)
     (effects (font (size 1.27 1.27)) (justify left bottom))
@@
     (effects (font (size 1.27 1.27)) (justify right bottom))
   )
+  (label "VSS" (at 146.05 67.31 180) (fields_autoplaced)
+    (effects (font (size 1.27 1.27)) (justify right bottom))
+  )
   (label "GPIO_05" (at 109.22 132.08 180) (fields_autoplaced)
     (effects (font (size 1.27 1.27)) (justify right bottom))
@@
     (effects (font (size 1.27 1.27)) (justify right bottom))
   )
+  (label "VSS" (at 157.48 72.39 0) (fields_autoplaced)
+    (effects (font (size 1.27 1.27)) (justify left bottom))
+  )
   (label "GPIO_04" (at 93.98 95.25 180) (fields_autoplaced)
     (effects (font (size 1.27 1.27)) (justify right bottom))
@@
     (effects (font (size 1.27 1.27)) (justify right bottom))
   )
+  (label "VDD" (at 157.48 74.93 0) (fields_autoplaced)
+    (effects (font (size 1.27 1.27)) (justify left bottom))
+  )
   (label "GPIO_00" (at 25.4 53.34 0) (fields_autoplaced)
     (effects (font (size 1.27 1.27)) (justify left bottom))
@@
     (effects (font (size 1.27 1.27)) (justify left bottom))
   )
+  (label "OSC_EN" (at 146.05 64.77 180) (fields_autoplaced)
+    (effects (font (size 1.27 1.27)) (justify right bottom))
+  )
   (label "VSS" (at 144.78 179.07 180) (fields_autoplaced)
     (effects (font (size 1.27 1.27)) (justify right bottom))
@@
     (effects (font (size 1.27 1.27)) (justify left bottom))
   )
+  (label "VSS" (at 149.86 58.42 180) (fields_autoplaced)
+    (effects (font (size 1.27 1.27)) (justify right bottom))
+  )
   (label "GPIO_03" (at 93.98 97.79 180) (fields_autoplaced)
     (effects (font (size 1.27 1.27)) (justify right bottom))
@@
     (effects (font (size 1.27 1.27)) (justify left bottom))
   )
+  (label "OSC_OUT" (at 161.29 67.31 0) (fields_autoplaced)
+    (effects (font (size 1.27 1.27)) (justify left bottom))
+  )
   (label "GPIO_02" (at 25.4 58.42 0) (fields_autoplaced)
     (effects (font (size 1.27 1.27)) (justify left bottom))
   )
+  (label "GPIO_23" (at 119.38 172.72 0) (fields_autoplaced)
+    (effects (font (size 1.27 1.27)) (justify left bottom))
+  )
   (label "TCK" (at 25.4 40.64 0) (fields_autoplaced)
     (effects (font (size 1.27 1.27)) (justify left bottom))
@@
     (effects (font (size 1.27 1.27)) (justify left bottom))
   )
+  (label "OSC_OUT" (at 109.22 172.72 180) (fields_autoplaced)
+    (effects (font (size 1.27 1.27)) (justify right bottom))
+  )
   (label "GPIO_24" (at 93.98 87.63 180) (fields_autoplaced)
     (effects (font (size 1.27 1.27)) (justify right bottom))
@@
     (effects (font (size 1.27 1.27)) (justify right bottom))
   )
+  (label "VDD" (at 161.29 64.77 0) (fields_autoplaced)
+    (effects (font (size 1.27 1.27)) (justify left bottom))
+  )
   (label "VREFP" (at 116.84 43.18 0) (fields_autoplaced)
     (effects (font (size 1.27 1.27)) (justify left bottom))
@@
   (label "GPIO_21" (at 99.06 120.65 180) (fields_autoplaced)
     (effects (font (size 1.27 1.27)) (justify right bottom))
+  )
+  (label "VDD" (at 157.48 58.42 0) (fields_autoplaced)
+    (effects (font (size 1.27 1.27)) (justify left bottom))
   )
   (label "VSS" (at 106.68 54.61 180) (fields_autoplaced)
@@
     )
   )
+  (symbol (lib_id "Device:C") (at 153.67 58.42 90) (unit 1)
+    (in_bom yes) (on_board yes) (dnp no)
+    (property "Reference" "C11" (at 152.4 59.69 90)
+      (effects (font (size 1.27 1.27)) (justify left))
+    )
+    (property "Value" "1u" (at 157.48 59.69 90)
+      (effects (font (size 1.27 1.27)) (justify left))
+    )
+    (property "Footprint" "SquantorCapacitor:C_0603" (at 157.48 57.4548 0)
+      (effects (font (size 1.27 1.27)) hide)
+    )
+    (property "Datasheet" "~" (at 153.67 58.42 0)
+      (effects (font (size 1.27 1.27)) hide)
+    )
+    (pin "1")
+    (pin "2")
+    (instances
+      (project "nuclone_LPC804M101DH24"
+        (path "/937928d4-4dfb-4f2f-91d0-697ec54ac283/00000000-0000-0000-0000-00006127a958"
+          (reference "C11") (unit 1)
+        )
+      )
+    )
+  )
   (symbol (lib_id "Device:FerriteBead") (at 113.03 34.29 90) (unit 1)
     (in_bom yes) (on_board yes) (dnp no)
@@
         (path "/937928d4-4dfb-4f2f-91d0-697ec54ac283/00000000-0000-0000-0000-00006127a958"
           (reference "C8") (unit 1)
+        )
+      )
+    )
+  )
+  (symbol (lib_id "Device:R") (at 153.67 74.93 90) (unit 1)
+    (in_bom yes) (on_board yes) (dnp no)
+    (property "Reference" "R11" (at 148.59 76.2 90)
+      (effects (font (size 1.27 1.27)))
+    )
+    (property "Value" "10K" (at 153.67 74.93 90)
+      (effects (font (size 1.27 1.27)))
+    )
+    (property "Footprint" "SquantorResistor:R_0603_hand" (at 153.67 76.708 90)
+      (effects (font (size 1.27 1.27)) hide)
+    )
+    (property "Datasheet" "~" (at 153.67 74.93 0)
+      (effects (font (size 1.27 1.27)) hide)
+    )
+    (pin "2")
+    (pin "1")
+    (instances
+      (project "nuclone_LPC804M101DH24"
+        (path "/937928d4-4dfb-4f2f-91d0-697ec54ac283/00000000-0000-0000-0000-00006127a958"
+          (reference "R11") (unit 1)
         )
       )
@@
     )
   )
+  (symbol (lib_id "SquantorGenericDigital:OSC_3state") (at 153.67 66.04 0) (unit 1)
+    (in_bom yes) (on_board yes) (dnp no)
+    (property "Reference" "U4" (at 153.67 62.23 0)
+      (effects (font (size 1.27 1.27)))
+    )
+    (property "Value" "TBD" (at 153.67 69.85 0)
+      (effects (font (size 1.27 1.27)))
+    )
+    (property "Footprint" "SquantorCrystal:Crystal_3225_4_hand" (at 153.67 66.04 0)
+      (effects (font (size 1.27 1.27)) hide)
+    )
+    (property "Datasheet" "" (at 153.67 66.04 0)
+      (effects (font (size 1.27 1.27)) hide)
+    )
+    (pin "3")
+    (pin "4")
+    (pin "1")
+    (pin "2")
+    (instances
+      (project "nuclone_LPC804M101DH24"
+        (path "/937928d4-4dfb-4f2f-91d0-697ec54ac283/00000000-0000-0000-0000-00006127a958"
+          (reference "U4") (unit 1)
+        )
+      )
+    )
+  )
   (symbol (lib_id "SquantorGenericAnalog:reference_sot23-3") (at 153.67 41.91 0) (unit 1)
     (in_bom yes) (on_board yes) (dnp no)
@@
     )
   )
+  (symbol (lib_id "SquantorSpecial:Solderjumper_2way_noconn") (at 114.3 172.72 0) (unit 1)
+    (in_bom yes) (on_board yes) (dnp no)
+    (property "Reference" "JP5" (at 114.3 168.91 0)
+      (effects (font (size 1.27 1.27)))
+    )
+    (property "Value" "OSC to GPIO_01" (at 114.3 176.53 0)
+      (effects (font (size 1.27 1.27)))
+    )
+    (property "Footprint" "SquantorSpecial:solder_jumper_0402_2way_noconn" (at 114.3 172.72 0)
+      (effects (font (size 1.27 1.27)) hide)
+    )
+    (property "Datasheet" "" (at 114.3 172.72 0)
+      (effects (font (size 1.27 1.27)) hide)
+    )
+    (pin "1")
+    (pin "2")
+    (instances
+      (project "nuclone_LPC804M101DH24"
+        (path "/937928d4-4dfb-4f2f-91d0-697ec54ac283/00000000-0000-0000-0000-00006127a958"
+          (reference "JP5") (unit 1)
+        )
+      )
+    )
+  )
   (symbol (lib_id "SquantorSpecial:Solderjumper_2way_noconn") (at 114.3 152.4 0) (unit 1)
     (in_bom yes) (on_board yes) (dnp no)
@@
         )
       )
+    )
+  )
+  (symbol (lib_id "Device:R") (at 153.67 72.39 90) (unit 1)
+    (in_bom yes) (on_board yes) (dnp no)
+    (property "Reference" "R10" (at 148.59 73.66 90)
+      (effects (font (size 1.27 1.27)))
+    )
+    (property "Value" "10K" (at 153.67 72.39 90)
+      (effects (font (size 1.27 1.27)))
+    )
+    (property "Footprint" "SquantorResistor:R_0603_hand" (at 153.67 74.168 90)
+      (effects (font (size 1.27 1.27)) hide)
+    )
+    (property "Datasheet" "~" (at 153.67 72.39 0)
+      (effects (font (size 1.27 1.27)) hide)
+    )
+    (pin "2")
+    (pin "1")
+    (instances
+      (project "nuclone_LPC804M101DH24"
+        (path "/937928d4-4dfb-4f2f-91d0-697ec54ac283/00000000-0000-0000-0000-00006127a958"
+          (reference "R10") (unit 1)
+        )
+      )
