File: electronics/nuclone_LPC845M301BD48_medium/nuclone_LPC845M301BD48_medium.kicad_sch (KiCad schematic)
At the start: 37 parts, among them J1 JTAG_2X05, J2 TYPE-C-31-M-12, J3 nuclone_medium_left, J4 nuclone_medium_right, SW1 RESET, SW2 Bootloader, U1 MCP1702-3.3V

Commit message: updated versions, fixed DRC's
Parts:
- N2: value V20240606 -> V20240628
- N4: value NuClone Medium template V1.5.1 -> NuClone LPC845 PQFP48
Changed lines of the file:
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@@
       (effects (font (size 1.524 1.524)) (justify left))
     )
-    (property "Value" "V20240606" (at 17.78 182.88 0)
+    (property "Value" "V20240628" (at 17.78 182.88 0)
       (effects (font (size 1.524 1.524)) (justify left))
     )
@@
       (effects (font (size 1.524 1.524)) (justify left))
     )
-    (property "Value" "NuClone Medium template V1.5.1" (at 20.32 170.18 0)
-      (effects (font (size 1.524 1.524)) (justify left))
-    )
+    (property "Value" "NuClone LPC845 PQFP48" (at 20.32 170.18 0)
+      (effects (font (size 1.524 1.524)) (justify left))
+    )

Commit message: prepped for production with updated versionnumbers and some minor changes
Parts:
- N2: value V20240628 -> V20240712
Changed lines of the file:
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@@
       (effects (font (size 1.524 1.524)) (justify left))
     )
-    (property "Value" "V20240628" (at 17.78 182.88 0)
+    (property "Value" "V20240712" (at 17.78 182.88 0)
       (effects (font (size 1.524 1.524)) (justify left))
     )
